Commit message: lastest stable version

File: foot_platform_ros/urdf/right/foot_platform.joints.xacro (robot description, xacro)
@@ -49,5 +49,5 @@
       <parent link="roll"/>
       <child link="yaw"/>
-      <limit effort="7" velocity="10.0" lower="${radians(-120)}" upper="${radians(120)}"/>
+      <limit effort="7" velocity="10.0" lower="${radians(-100)}" upper="${radians(100)}"/>
       <axis xyz="0 0 1"/>
     </joint>

File: foot_platform_ros/urdf/right/foot_platform.links.xacro (robot description, xacro)
@@ -124,5 +124,5 @@
         <inertial>
         <origin xyz="-0.03198766 0.00021421 0.02133190" rpy="0 0 0"/>
-        <mass value="0.37200000"/><!-- 0.372 kg -->
+        <mass value="0.30000000"/><!-- 0.372 kg -->
         <inertia ixx="0.00044045"  ixy="-0.00001582"  ixz="0.00271438" iyy="-0.00000105" iyz="-0.00000105" izz="0.00282256" />
       </inertial>
