Commit message: backup 4.02.2021

File: foot_platform_ros/urdf/left/foot_platform.joints.xacro (robot description, xacro)
@@ -11,64 +11,64 @@
   <xacro:property name="d7_platform" value="${platform_geom_data['d7']}"/> <!-- [m]-->
   <xacro:property name="r8_platform" value="${platform_geom_data['r8']}"/> <!-- [m]-->
-  <xacro:macro name="define_platform_joints">
-    <joint name="platform_y" type="prismatic">
+  <xacro:macro name="define_platform_joints" params="platform_id:=left">
+    <joint name="${platform_id}_platform_y" type="prismatic">
       <origin xyz="0 0 0" rpy="-${pi/2} 0 0"/>
-      <parent link="platform_base_link"/>
-      <child link="y"/>
+      <parent link="${platform_id}_platform_base_link"/>
+      <child link="${platform_id}_platform_y"/>
       <limit effort="23.5" velocity="10.0" lower="-0.090" upper="0.090"/>
       <axis xyz="0 0 1"/>
     </joint>
-    <joint name="platform_x" type="prismatic">
+    <joint name="${platform_id}_platform_x" type="prismatic">
       <origin xyz="0 0 0" rpy="${pi/2} 0 ${pi/2}"/>
-      <parent link="y"/>
-      <child link="x"/>
+      <parent link="${platform_id}_platform_y"/>
+      <child link="${platform_id}_platform_x"/>
       <limit effort="30" velocity="10.0" lower="-0.0975" upper="0.0975"/>
       <axis xyz="0 0 1"/>
     </joint>
-    <joint name="z_joint" type="fixed">
+    <joint name="${platform_id}_z_joint" type="fixed">
       <origin xyz="0 0 0" rpy="0 0 ${pi}"/>
-      <parent link="x"/>
-      <child link="z_link"/>
+      <parent link="${platform_id}_platform_x"/>
+      <child link="${platform_id}_platform_z_link"/>
     </joint>
-    <joint name="platform_pitch" type="revolute">
+    <joint name="${platform_id}_platform_pitch" type="revolute">
       <origin xyz="${r3_platform} 0 0" rpy="0 0 0"/>
-      <parent link="z_link"/>
-      <child link="pitch"/>
+      <parent link="${platform_id}_platform_z_link"/>
+      <child link="${platform_id}_platform_pitch"/>
       <limit effort="7" velocity="10.0" lower="${radians(-27.5)}" upper="${radians(27.5)}"/>
       <axis xyz="0 0 1"/>
     </joint>
-    <joint name="platform_roll" type="revolute">
+    <joint name="${platform_id}_platform_roll" type="revolute">
       <origin xyz="0 0 0" rpy="${pi/2} 0 0"/>
-      <parent link="pitch"/>
-      <child link="roll"/>
-      <limit effort="7" velocity="10.0" lower="${radians(-20.5)}" upper="${radians(80)}"/>
+      <parent link="${platform_id}_platform_pitch"/>
+      <child link="${platform_id}_platform_roll"/>
+      <limit effort="7" velocity="10.0" lower="${radians(-20.5)}" upper="${radians(0)}"/>
       <axis xyz="0 0 1"/>
     </joint>
-    <joint name="platform_yaw" type="revolute">
+    <joint name="${platform_id}_platform_yaw" type="revolute">
       <origin xyz="0 0 0" rpy="-${pi/2} 0 -${pi/2}"/>
-      <parent link="roll"/>
-      <child link="yaw"/>
-      <limit effort="7" velocity="10.0" lower="${radians(-120)}" upper="${radians(120)}"/>
+      <parent link="${platform_id}_platform_roll"/>
+      <child link="${platform_id}_platform_yaw"/>
+      <limit effort="7" velocity="10.0" lower="${radians(-25)}" upper="${radians(25)}"/>
       <axis xyz="0 0 1"/>
     </joint>
-    <joint name="fSensor_joint" type="fixed">
+    <joint name="${platform_id}_fSensor_joint" type="fixed">
       <origin xyz="0 0 ${d6_platform}" rpy="0 0 ${pi/2}"/>
-      <parent link="yaw"/>
-      <child link="fSensor"/>
+      <parent link="${platform_id}_platform_yaw"/>
+      <child link="${platform_id}_platform_fSensor"/>
     </joint>
-    <joint name="footRest_joint" type="fixed">
+    <joint name="${platform_id}_footRest_joint" type="fixed">
       <origin xyz="0 0 ${d7_platform}" rpy="0 0 ${pi}"/>
-      <parent link="fSensor"/>
-      <child link="foot_rest"/>
+      <parent link="${platform_id}_platform_fSensor"/>
+      <child link="${platform_id}_platform_foot_rest"/>
     </joint>
-    <joint name="virtualAnkle_joint" type="fixed">
+    <joint name="${platform_id}_virtualAnkle_joint" type="fixed">
       <origin xyz="${-r7_leg} 0 ${d7_leg}" rpy="0 0 0"/>
-      <parent link="foot_rest"/>
-      <child link="virtual_ankle"/>
+      <parent link="${platform_id}_platform_foot_rest"/>
+      <child link="${platform_id}_platform_virtual_ankle"/>
     </joint>
-    <joint name="footTip_joint" type="fixed">
+    <joint name="${platform_id}_footTip_joint" type="fixed">
       <origin xyz="${r8_platform} 0 0" rpy="0 0 0"/>
-      <parent link="foot_rest"/>
-      <child link="pedal_tip"/>
+      <parent link="${platform_id}_platform_foot_rest"/>
+      <child link="${platform_id}_platform_pedal_tip"/>
     </joint>
 </xacro:macro>

File: foot_platform_ros/urdf/left/foot_platform.links.xacro (robot description, xacro)
@@ -5,6 +5,6 @@
   <xacro:property name="pitch_gear_r" value="${12.0}"/>
   <xacro:property name="roll_yaw_gear_r" value="${12.96}"/>
-  <xacro:macro name="define_platform_links">
-    <link name="platform_base_link" >
+  <xacro:macro name="define_platform_links" params="platform_id:=left">
+    <link name="${platform_id}_platform_base_link" >
       <!--inertial>  KDL doesn't like the base with inertia
         <mass value="6.20696344"/>
@@ -25,5 +25,5 @@
       </collision>
     </link>
-    <link name="y">
+    <link name="${platform_id}_platform_y">
         <inertial>
         <origin xyz="-0.02817123 -0.07585496 0.00969366" rpy="0 0 0"/>
@@ -44,5 +44,5 @@
       </collision>
     </link>
-    <link name="x">
+    <link name="${platform_id}_platform_x">
       <inertial>
         <origin xyz="-0.15354810 -0.02479498 -0.06831312" rpy="0 0 0"/>
@@ -63,6 +63,6 @@
       </collision>
     </link>
-    <link name="z_link"/> <!--virtual link-->
-    <link name="pitch">
+    <link name="${platform_id}_platform_z_link"/> <!--virtual link-->
+    <link name="${platform_id}_platform_pitch">
       <inertial>
         <origin xyz="-0.00593072	-0.00000124	 -0.00156324" rpy="0 0 0"/>
@@ -83,5 +83,5 @@
       </collision>
     </link>
-    <link name="roll">
+    <link name="${platform_id}_platform_roll">
       <inertial>
         <origin xyz="0.03719409 -0.00002562 -0.00002217" rpy="0 0 0"/>
@@ -102,5 +102,5 @@
       </collision>
     </link>
-    <link name="yaw">
+    <link name="${platform_id}_platform_yaw">
       <inertial>
         <origin xyz="-0.00002617   0.00000265  0.10239610" rpy="0 0 0"/>
@@ -121,5 +121,5 @@
       </collision>
     </link>
-    <link name="fSensor">
+    <link name="${platform_id}_platform_fSensor">
         <inertial>
         <origin xyz="-0.03198766 0.00021421 0.02133190" rpy="0 0 0"/>
@@ -140,7 +140,7 @@
       </collision>
     </link>
-    <link name="foot_rest" /> <!-- virtual link-->
-    <link name="virtual_ankle" /> <!-- virtual link-->
-    <link name="pedal_tip" /> <!-- virtual link-->
+    <link name="${platform_id}_platform_foot_rest" /> <!-- virtual link-->
+    <link name="${platform_id}_platform_virtual_ankle" /> <!-- virtual link-->
+    <link name="${platform_id}_platform_pedal_tip" /> <!-- virtual link-->
   </xacro:macro>
 </robot>

File: foot_platform_ros/urdf/right/foot_platform.joints.xacro (robot description, xacro)
@@ -11,64 +11,64 @@
   <xacro:property name="d7_platform" value="${platform_geom_data['d7']}"/> <!-- [m]-->
   <xacro:property name="r8_platform" value="${platform_geom_data['r8']}"/> <!-- [m]-->
-  <xacro:macro name="define_platform_joints">
-    <joint name="platform_y" type="prismatic">
+  <xacro:macro name="define_platform_joints" params="platform_id:=right">
+    <joint name="${platform_id}_platform_y" type="prismatic">
       <origin xyz="0 0 0" rpy="-${pi/2} 0 0"/>
-      <parent link="platform_base_link"/>
-      <child link="y"/>
+      <parent link="${platform_id}_platform_base_link"/>
+      <child link="${platform_id}_platform_y"/>
       <limit effort="23.5" velocity="10.0" lower="-0.090" upper="0.090"/>
       <axis xyz="0 0 1"/>
     </joint>
-    <joint name="platform_x" type="prismatic">
+    <joint name="${platform_id}_platform_x" type="prismatic">
       <origin xyz="0 0 0" rpy="${pi/2} 0 ${pi/2}"/>
-      <parent link="y"/>
-      <child link="x"/>
+      <parent link="${platform_id}_platform_y"/>
+      <child link="${platform_id}_platform_x"/>
       <limit effort="30" velocity="10.0" lower="-0.0975" upper="0.0975"/>
       <axis xyz="0 0 1"/>
     </joint>
-    <joint name="z_joint" type="fixed">
+    <joint name="${platform_id}_z_joint" type="fixed">
       <origin xyz="0 0 0" rpy="0 0 ${pi}"/>
-      <parent link="x"/>
-      <child link="z_link"/>
+      <parent link="${platform_id}_platform_x"/>
+      <child link="${platform_id}_platform_z_link"/>
     </joint>
-    <joint name="platform_pitch" type="revolute">
+    <joint name="${platform_id}_platform_pitch" type="revolute">
       <origin xyz="${r3_platform} 0 0" rpy="0 0 0"/>
-      <parent link="z_link"/>
-      <child link="pitch"/>
+      <parent link="${platform_id}_platform_z_link"/>
+      <child link="${platform_id}_platform_pitch"/>
       <limit effort="7" velocity="10.0" lower="${radians(-27.5)}" upper="${radians(27.5)}"/>
       <axis xyz="0 0 1"/>
     </joint>
-    <joint name="platform_roll" type="revolute">
+    <joint name="${platform_id}_platform_roll" type="revolute">
       <origin xyz="0 0 0" rpy="${pi/2} 0 0"/>
-      <parent link="pitch"/>
-      <child link="roll"/>
-      <limit effort="7" velocity="10.0" lower="${radians(-80)}" upper="${radians(20.5)}"/>
+      <parent link="${platform_id}_platform_pitch"/>
+      <child link="${platform_id}_platform_roll"/>
+      <limit effort="7" velocity="10.0" lower="${radians(0.0)}" upper="${radians(20.5)}"/>
       <axis xyz="0 0 1"/>
     </joint>
-    <joint name="platform_yaw" type="revolute">
+    <joint name="${platform_id}_platform_yaw" type="revolute">
       <origin xyz="0 0 0" rpy="-${pi/2} 0 -${pi/2}"/>
-      <parent link="roll"/>
-      <child link="yaw"/>
-      <limit effort="7" velocity="10.0" lower="${radians(-100)}" upper="${radians(100)}"/>
+      <parent link="${platform_id}_platform_roll"/>
+      <child link="${platform_id}_platform_yaw"/>
+      <limit effort="7" velocity="10.0" lower="${radians(-25)}" upper="${radians(25)}"/>
       <axis xyz="0 0 1"/>
     </joint>
-    <joint name="fSensor_joint" type="fixed">
+    <joint name="${platform_id}_fSensor_joint" type="fixed">
       <origin xyz="0 0 ${d6_platform}" rpy="0 0 ${pi/2}"/>
-      <parent link="yaw"/>
-      <child link="fSensor"/>
+      <parent link="${platform_id}_platform_yaw"/>
+      <child link="${platform_id}_platform_fSensor"/>
     </joint>
-    <joint name="footRest_joint" type="fixed">
+    <joint name="${platform_id}_footRest_joint" type="fixed">
       <origin xyz="0 0 ${d7_platform}" rpy="0 0 ${pi}"/>
-      <parent link="fSensor"/>
-      <child link="foot_rest"/>
+      <parent link="${platform_id}_platform_fSensor"/>
+      <child link="${platform_id}_platform_foot_rest"/>
     </joint>
-    <joint name="virtualAnkle_joint" type="fixed">
+    <joint name="${platform_id}_virtualAnkle_joint" type="fixed">
       <origin xyz="${-r7_leg} 0 ${d7_leg}" rpy="0 0 0"/>
-      <parent link="foot_rest"/>
-      <child link="virtual_ankle"/>
+      <parent link="${platform_id}_platform_foot_rest"/>
+      <child link="${platform_id}_platform_virtual_ankle"/>
     </joint>
-    <joint name="footTip_joint" type="fixed">
+    <joint name="${platform_id}_footTip_joint" type="fixed">
       <origin xyz="${r8_platform} 0 0" rpy="0 0 0"/>
-      <parent link="foot_rest"/>
-      <child link="pedal_tip"/>
+      <parent link="${platform_id}_platform_foot_rest"/>
+      <child link="${platform_id}_platform_pedal_tip"/>
     </joint>
 </xacro:macro>

File: foot_platform_ros/urdf/right/foot_platform.links.xacro (robot description, xacro)
@@ -5,6 +5,6 @@
   <xacro:property name="pitch_gear_r" value="${12.0}"/>
   <xacro:property name="roll_yaw_gear_r" value="${12.96}"/>
-  <xacro:macro name="define_platform_links">
-    <link name="platform_base_link" >
+  <xacro:macro name="define_platform_links" params="platform_id:=right">
+    <link name="${platform_id}_platform_base_link" >
       <!--inertial>  KDL doesn't like the base with inertia
         <mass value="6.20696344"/>
@@ -25,5 +25,5 @@
       </collision>
     </link>
-    <link name="y">
+    <link name="${platform_id}_platform_y">
         <inertial>
         <origin xyz="0.02817123 -0.07585496 -0.00969366" rpy="0 0 0"/>
@@ -44,5 +44,5 @@
       </collision>
     </link>
-    <link name="x">
+    <link name="${platform_id}_platform_x">
       <inertial>
         <origin xyz="-0.15354818 0.02479469 0.08202519" rpy="0 0 0"/>
@@ -63,6 +63,6 @@
       </collision>
     </link>
-    <link name="z_link"/> <!--virtual link-->
-    <link name="pitch">
+    <link name="${platform_id}_platform_z_link"/> <!--virtual link-->
+    <link name="${platform_id}_platform_pitch">
       <inertial>
         <origin xyz="-0.00510491 0.00000315  0.00119335" rpy="0 0 0"/>
@@ -83,5 +83,5 @@
       </collision>
     </link>
-    <link name="roll">
+    <link name="${platform_id}_platform_roll">
       <inertial>
         <origin xyz="0.03719409 -0.00002562 -0.00002217" rpy="0 0 0"/>
@@ -102,5 +102,5 @@
       </collision>
     </link>
-    <link name="yaw">
+    <link name="${platform_id}_platform_yaw">
       <inertial>
         <origin xyz="0.00002617   -0.00000265 0.10239610" rpy="0 0 0"/>
@@ -121,5 +121,5 @@
       </collision>
     </link>
-    <link name="fSensor">
+    <link name="${platform_id}_platform_fSensor">
         <inertial>
         <origin xyz="-0.03198766 0.00021421 0.02133190" rpy="0 0 0"/>
@@ -140,7 +140,7 @@
       </collision>
     </link>
-    <link name="foot_rest" /> <!-- virtual link-->
-    <link name="virtual_ankle" /> <!-- virtual link-->
-    <link name="pedal_tip" /> <!-- virtual link-->
+    <link name="${platform_id}_platform_foot_rest" /> <!-- virtual link-->
+    <link name="${platform_id}_platform_virtual_ankle" /> <!-- virtual link-->
+    <link name="${platform_id}_platform_pedal_tip" /> <!-- virtual link-->
   </xacro:macro>
 </robot>

File: foot_platform_ros/urdf/right/foot_platform.urdf.xacro (robot description, xacro)
@@ -1,5 +1,5 @@
 <?xml version="1.0"?>
 <robot name="foot_platform" xmlns:xacro="http://www.ros.org/wiki/xacro">
- <xacro:macro name="create_platform">
+<xacro:macro name="create_platform">
     <xacro:include filename="$(find foot_platform_ros)/urdf/right/foot_platform.links.xacro"/>
     <xacro:include filename="$(find foot_platform_ros)/urdf/right/foot_platform.joints.xacro"/>

Commit message: fixed bug with unrecognized platform

File: foot_platform_ros/urdf/left/foot_platform.joints.xacro (robot description, xacro)
@@ -42,5 +42,5 @@
       <parent link="${platform_id}_platform_pitch"/>
       <child link="${platform_id}_platform_roll"/>
-      <limit effort="7" velocity="10.0" lower="${radians(-20.5)}" upper="${radians(0)}"/>
+      <limit effort="7" velocity="10.0" lower="${radians(-20.5)}" upper="${radians(20.5)}"/>
       <axis xyz="0 0 1"/>
     </joint>

File: foot_platform_ros/urdf/right/foot_platform.joints.xacro (robot description, xacro)
@@ -42,5 +42,5 @@
       <parent link="${platform_id}_platform_pitch"/>
       <child link="${platform_id}_platform_roll"/>
-      <limit effort="7" velocity="10.0" lower="${radians(0.0)}" upper="${radians(20.5)}"/>
+      <limit effort="7" velocity="10.0" lower="${radians(-20.5)}" upper="${radians(20.5)}"/>
       <axis xyz="0 0 1"/>
     </joint>

Commit message: update params virtual wall and foot state publisher

File: foot_platform_ros/urdf/left/foot_platform.joints.xacro (robot description, xacro)
@@ -42,5 +42,5 @@
       <parent link="${platform_id}_platform_pitch"/>
       <child link="${platform_id}_platform_roll"/>
-      <limit effort="7" velocity="10.0" lower="${radians(-20.5)}" upper="${radians(20.5)}"/>
+      <limit effort="7" velocity="10.0" lower="${radians(-20.5)}" upper="${radians(0)}"/>
       <axis xyz="0 0 1"/>
     </joint>

File: foot_platform_ros/urdf/right/foot_platform.joints.xacro (robot description, xacro)
@@ -42,5 +42,5 @@
       <parent link="${platform_id}_platform_pitch"/>
       <child link="${platform_id}_platform_roll"/>
-      <limit effort="7" velocity="10.0" lower="${radians(-20.5)}" upper="${radians(20.5)}"/>
+      <limit effort="7" velocity="10.0" lower="${radians(0.0)}" upper="${radians(20.5)}"/>
       <axis xyz="0 0 1"/>
     </joint>
